File: aeroly_pro3.kicad_sch (KiCad schematic)
At the start: 75 parts, among them J1 B2B-PH-K-S_LF__SN_, J2 TYPE-C-31-M-12, P1 AFC30-S12FCC-00, SW1 TSB001A3818A, SW2 TSB001A3818A, SW3 TSB001A3818A, SW4 TSB001A3818A, U1 ESP32-S3-MINI-1, U10 SGP40-D-R4, U11 BMP390L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

Commit message: Add files via upload
Parts:
- R22: value 1.18K -> 100
Other:
- note added: "used 1.18k for R22 in the prototype 2"
Changed lines of the file:
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@@
 		)
 	)
+	(text "used 1.18k for R22\nin the prototype 2"
+		(exclude_from_sim no)
+		(at 221.742 31.75 0)
+		(effects
+			(font
+				(size 1.27 1.27)
+			)
+		)
+	)
 	(text "ILIM Set by an external \nresistor from ILIM \nto VSS"
 		(exclude_from_sim no)
@@
 			)
 		)
-		(property "Value" "1.18K"
+		(property "Value" "100"
 			(at 214.376 36.576 0)
 			(effects
